File: ErgoDOX pcb/ErgoDOX.kicad_pcb (KiCad board)
At the start: 2 copper layers, 182.8 x 158.9 mm, 76 parts, among them J1 USB, J2 3.5mm, J3 JMP, J4 JMP, SW0:10 SW0:3, SW0:11 SW0:2, SW0:12 SW0:1, SW0:7 SW0:6, SW0:8 SW0:5, SW0:9 SW0:4, SW1:10 SW1:3, SW1:11 SW1:2, SW1:12 SW1:1, SW1:13 SW1:0, SW1:9 SW1:4, SW2:10 SW2:3, SW2:11 SW2:2, SW2:12 SW2:1, SW2:13 SW2:0, SW2:7 SW2:6, SW2:8 SW2:5, SW2:9 SW2:4, SW3:10 SW3:3, SW3:11 SW3:2, SW3:12 SW3:1, SW3:13 SW3:0, SW3:8 SW3:5, SW3:9 SW3:4, SW4:10 SW4:3, SW4:11 SW4:2, SW4:12 SW4:1, SW4:13 SW4:0, SW4:7 SW4:6, SW4:8 SW4:5, SW4:9 SW4:4, SW5:10 SW5:3, SW5:11 SW5:2, SW5:12 SW5:1, SW5:13 SW5:0, SW5:7 SW5:6, SW5:8 SW5:5, SW5:9 SW5:4, U1 TEENSY2.0, U2 MCP23018

Commit message: Long overdue update to the board.
Parts:
- removed D1:7, D1:8: D, DIODE
- removed H99: MECHANICAL, ErgoDOXmech
- removed JP1, JP2: JUMPER, GAP
- removed LED_A1: LEDa, MX_LED
- removed LED_B1: LEDb, MX_LED
- removed LED_C1: LEDc, MX_LED
- removed RA1: LEDa, RESISTOR
- removed RB1: LEDb, RESISTOR
- removed RC1: LEDc, RESISTOR
- removed S1, S2: STAB200, STAB_PCB940
- removed STAR_1: STAR_FRONT, ErgoDOX pcb:STAR
- removed STAR_2: STAR_BACK, ErgoDOX pcb:STAR
- removed STITCHING_VIA (x11): ~, lib_footprints:STITCHING_VIA
- removed SW4:8: SW4:5, ErgoDOX pcb:MX_FLIP_DIODE
- removed SW5:10: SW5:3, ErgoDOX pcb:MX_FLIP_DIODE
- removed SW5:11: SW5:2, ErgoDOX pcb:MX_FLIP_DIODE
- removed SW5:12: SW5:1, ErgoDOX pcb:MX_FLIP_DIODE
- removed SW5:13: SW5:0, ErgoDOX pcb:MX_FLIP_XX
- removed SW5:7: SW5:6, ErgoDOX pcb:MX_FLIP_DIODE
- removed SW5:8: SW5:5, ErgoDOX pcb:MX_FLIP_DIODE
- removed SW5:9: SW5:4, ErgoDOX pcb:MX_FLIP_DIODE
- removed SX0:10: SX0:3, MX_FLIP
- removed SX0:11: SX0:2, MX_FLIP
- removed SX1:7: SX1:6, MX_FLIP
- removed SX1:8: SX1:5, MX_FLIP
- removed U2: MCP23018, DIP28_300
- added C1: 32pF, Capacitors_SMD:C_0805_HandSoldering, B.Cu at (161.0, 146.6)
- added C2: 32pF, Capacitors_SMD:C_0805_HandSoldering, B.Cu at (161.0, 154.2)
- added C3: 1uF, Capacitors_SMD:C_0805_HandSoldering, B.Cu at (140.3, 138.7)
- added C4: 1uF, Capacitors_SMD:C_0805_HandSoldering, B.Cu at (146.6, 156.5)
- added C5: 1uF, Capacitors_SMD:C_0805_HandSoldering, B.Cu at (132.1, 152.7)
- added C6: 1uF, Capacitors_SMD:C_0805_HandSoldering, B.Cu at (132.6, 142.0)
- added C7: 1uF, Capacitors_SMD:C_0805_HandSoldering, B.Cu at (152.9, 143.3)
- added C8: 1uF, Capacitors_SMD:C_0805_HandSoldering, B.Cu at (140.3, 136.7)
- added C9: 1uF, Capacitors_SMD:C_0805_HandSoldering, F.Cu at (187.5, 152.9)
- added IC1: ATMEGA32U4, Housings_QFP:TQFP-44_10x10mm_Pitch0.8mm, B.Cu at (142.0, 147.3)
- added R3: 22, Resistors_SMD:R_0805_HandSoldering, F.Cu at (163.1, 138.7)
- added R4: 22, Resistors_SMD:R_0805_HandSoldering, F.Cu at (163.1, 141.5)
- added R5: 1k, Resistors_SMD:R_0805_HandSoldering, B.Cu at (136.7, 155.7)
- added SW0:13: SW0:0, footprints:MX_FLIP_DIODE_mod, F.Cu at (190.5, 133.3)
- added SW1:7: SW1:6, footprints:MX_FLIP_DIODE_mod, F.Cu at (95.2, 133.3)
- added SW1:8: SW1:5, footprints:MX_FLIP_DIODE_mod, F.Cu at (114.3, 111.9)
- added SW3:7: SW3:6, footprints:MX_FLIP_DIODE_mod, F.Cu at (95.2, 92.9)
- added X1: XTAL, Crystals:Crystal_HC49-U_Vertical, B.Cu at (156.7, 148.1)
- J1: value USB -> JMP; footprint USBMINImod -> footprints:100PITCH1X3
- J2: value 3.5mm -> USB_mini_micro_B; footprint 4pin35mmAudio -> footprints:USBMINI
- J3: value JMP -> 3.5mm; footprint 100PITCH1X3 -> footprints:4pin35mmAudio
- J4: footprint 100PITCH1X3 -> footprints:100PITCH1X3; moved to B.Cu
- R1, R2: footprint RESISTOR -> Resistors_SMD:R_0805_HandSoldering
- SW0:10, SW0:11, SW0:12, SW0:7, SW0:8, SW0:9, SW1:10, SW1:11, SW1:12, SW1:13, SW1:9, SW2:10, SW2:11, SW2:12, SW2:7, SW2:8, SW2:9, SW3:10, SW3:11, SW3:12, SW3:8, SW3:9, SW4:10, SW4:11, SW4:12, SW4:7, SW4:9: footprint ErgoDOX pcb:MX_FLIP_DIODE -> footprints:MX_FLIP_DIODE_mod
- SW2:13, SW3:13, SW4:13: footprint ErgoDOX pcb:MX_FLIP_XX -> footprints:MX_FLIP_DIODE_mod
- U1: value TEENSY2.0 -> MCP23018-SSOP; footprint TEENSY_2.0 -> Housings_SSOP:SSOP-24_5.3x8.2mm_Pitch0.65mm; moved to B.Cu
- moved SW0:12 130.3 mm to (171.4, 128.6), turned to 0 degrees
- moved J2 120.8 mm to (205.2, 51.6)
- moved U1 106.6 mm to (196.6, 147.1)
- moved SW0:11 95.0 mm to (152.4, 126.2), turned to 0 degrees
- moved SW0:9 72.3 mm to (114.3, 150.0), turned to 0 degrees
- moved SW0:8 62.5 mm to (114.3, 131.0), turned to 0 degrees
- moved SW0:7 61.2 mm to (95.2, 152.4), turned to 0 degrees
- moved SW0:10 57.5 mm to (133.3, 128.6), turned to 0 degrees
- moved J1 54.8 mm to (88.6, 55.1), turned to 90 degrees
- moved SW1:10 38.7 mm to (152.4, 107.2)
- moved SW2:10 38.7 mm to (152.4, 88.1)
- moved SW3:10 38.7 mm to (152.4, 69.1)
- moved SW1:9 38.1 mm to (133.3, 109.5)
- moved SW2:9 38.1 mm to (133.3, 90.5)
- moved SW3:9 38.1 mm to (133.3, 71.4)
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Connections:
- J1 pad 2: (no net) -> Net-(J1-Pad2)
- J1 pad 3: (no net) -> GND
- J2 pad 1: N-000003 -> VCC
- J2 pad 2: /SDAM -> Net-(J2-Pad2)
- J2 pad 3: /SCLM -> Net-(J2-Pad3)
- J2 pad 4: N-000001 -> (no net)
- J2 pad 5: /SCLM -> GND
- J2 pad 6: /SDAM -> GND
- J3 pad 1: VCC -> Net-(J1-Pad2)
- J3 pad 2: N-000003 -> /SDAM
- J3 pad 3: GND -> /SCLM
- J4 pad 2: N-000001 -> Net-(J3-Pad4)
- U1 pad 10: /COL1 -> VCC
- U1 pad 11: /COL0 -> /SCLM
- U1 pad 12: (no net) -> /SDAM
- U1 pad 18: GND -> (no net)
- U1 pad 2: /COL6 -> (no net)
- U1 pad 20: VCC -> (no net)
- U1 pad 21: /LED_A -> (no net)
- U1 pad 22: /LED_B -> (no net)
- U1 pad 23: /ROW0 -> (no net)
- U1 pad 24: /ROW1 -> (no net)
- U1 pad 3: /COL5 -> (no net)
- U1 pad 4: /COL4 -> (no net)
- U1 pad 5: /COL10 -> (no net)
- U1 pad 6: /LED_C -> (no net)
- U1 pad 7: /SCLM -> (no net)
- U1 pad 8: /SDAM -> (no net)
- U1 pad 9: /COL11 -> (no net)
Routing:
- net /ROW0: track 404.2 -> 140.8 mm
- net /ROW5: track 225.1 -> 0.00 mm
- net /COL11: track 316.5 -> 121.7 mm
- net /COL6: track 259.5 -> 83.6 mm
- net /COL5: track 225.8 -> 61.1 mm
- net VCC: track 160.4 -> 0.00 mm
- net /COL1: track 291.8 -> 134.3 mm
- net /ROW1: track 318.2 -> 161.9 mm
- net /COL4: track 274.3 -> 121.8 mm
- net N-000067: track 127.4 -> 0.00 mm
- net /SDAM: track 127.2 -> 0.00 mm
- net /COL10: track 233.7 -> 107.1 mm
- net /SCLM: track 119.8 -> 0.00 mm
- net N-000068: track 119.1 -> 0.00 mm
- net /ROW2: track 295.3 -> 182.7 mm
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- removed copper zone on B.Cu, net GND
- removed copper zone on F.Cu, net GND
Other:
- board outline removed
- net class Default: clearance 0.3048 -> 0.2286; trace_width 0.6 -> 0.254; via_dia 0.6096 -> 0.6; via_drill 0.508 -> 0.4
- rule pad_to_mask_clearance: 0.2032 -> 0.2
- rule trace_clearance: 0.3048 -> 0.2286
- rule trace_min: 0.0254 -> 0.2032
- rule via_min_drill: 0.2032 -> 0.254
- board text removed: "5V"
- board text removed: "Components are intended to be placed on the side they are drawn. It is however possible to invert the design. See the webpage for further instructions. www.ergodox.io"
- board text removed: "D+"
- board text removed: "D-"
- board text removed: "Design by Dominic Beauchamp, based on the Key64 by Nestor A. Diaz"
- board text removed: "Drawn in KiCAD by Fredrik Atmer, Bathroom Epiphanies"
- board text removed: "ErgoDox"
- board text removed: "FR4 Tg170° Laminate 24mil traces on 1oz copper"
- board text removed: "GND"
- board text removed: "ID"
- board text removed: "LEFT HAND"
- board text removed: "RIGHT HAND"
- board text removed: "Revision 11-18-2016 PendulumKB"
